File: pcb/antiflood.sch (KiCad schematic (older format))
At the start: 94 parts, among them J1 Barrel_Jack, J10 Screw_Terminal_01x02, J11 Screw_Terminal_01x02, J12 Screw_Terminal_01x02, J13 Screw_Terminal_01x02, J2 Conn_01x03_Male, J3 01x03, J4 01x03, J5 Conn_02x04_Odd_Even, J6 Conn_02x05_Odd_Even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

Commit message: PCB: tracking
Changed lines of the file:
@@
 Text Label 3250 3100 0    60   ~ 0
 DBG
-Text Label 3100 4900 0    60   ~ 0
+Text Label 3100 5200 0    60   ~ 0
 FON
 Text Label 3100 5000 0    60   ~ 0
@@
 Text Label 600  7200 0    60   ~ 0
 PON
+Text Label 3100 4900 0    60   ~ 0
+PCL
 Text Label 3100 5100 0    60   ~ 0
-PCL
-Text Label 3100 5200 0    60   ~ 0
 PON
 $Comp
