File: pcb/antiflood.kicad_pcb (KiCad board)
At the start: 2 copper layers, 88 x 84 mm, 98 parts, among them J1 Barrel_Jack, J10 Screw_Terminal_01x02, J11 Screw_Terminal_01x02, J12 Screw_Terminal_01x02, J13 Screw_Terminal_01x02, J2 Conn_01x03_Male, J3 01x03, J4 01x03, J5 Conn_02x04_Odd_Even, J6 Conn_02x05_Odd_Even, J7 Conn_02x03_Odd_Even, J8 Screw_Terminal_01x02, J9 Screw_Terminal_01x02, K1 P-5, K2 P-5, Q1 MMBT3904, Q2 MMBT3904, SW1 SW_Push, SW2 SW_Push, SW3 SW_Push, U1 ATMEGA328P-AU, U2 TL7705, U3 LM1117-3.3, U4 MT3608, U5 MC34063, U6 TP4056, Y1 16MHz

Commit message: PCB: before filling
Routing:
- net GND: track 15.7 -> 101.8 mm, vias 4 -> 44
- net +5V: track 340.4 -> 364.9 mm
- added copper zone on B.Cu, net GND
- added copper zone on F.Cu, net GND
Changed lines of the file:
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@@
   (general
     (links 217)
-    (no_connects 62)
+    (no_connects 61)
     (area 71.454999 50.924999 159.555001 135.025001)
     (thickness 1.6)
     (drawings 24)
-    (tracks 725)
+    (tracks 826)
     (zones 0)
     (modules 98)
@@
   (gr_line (start 159.505 50.975) (end 159.505 134.975) (angle 90) (layer Edge.Cuts) (width 0.1))
   (gr_line (start 71.505 50.975) (end 159.505 50.975) (angle 90) (layer Edge.Cuts) (width 0.1))
+  (segment (start 100.5 131) (end 100.5 129.5) (width 0.4) (layer F.Cu) (net 1))
+  (via (at 100.5 129.5) (size 0.6) (drill 0.4) (layers F.Cu B.Cu) (net 1))
+  (segment (start 100.5 132.5) (end 100.5 131) (width 0.4) (layer F.Cu) (net 1))
+  (via (at 100.5 131) (size 0.6) (drill 0.4) (layers F.Cu B.Cu) (net 1))
+  (segment (start 102.87 133.095) (end 101.095 133.095) (width 0.4) (layer F.Cu) (net 1) (status 400000))
+  (segment (start 101.095 133.095) (end 100.5 132.5) (width 0.4) (layer F.Cu) (net 1))
+  (via (at 100.5 132.5) (size 0.6) (drill 0.4) (layers F.Cu B.Cu) (net 1))
+  (segment (start 84.455 99.06) (end 84.455 98.455) (width 0.5) (layer F.Cu) (net 1) (status 400000))
+  (segment (start 84.455 98.455) (end 83.5 97.5) (width 0.5) (layer F.Cu) (net 1))
+  (via (at 83.5 97.5) (size 0.6) (drill 0.4) (layers F.Cu B.Cu) (net 1))
+  (segment (start 76.2 99.06) (end 76.2 98.2) (width 0.5) (layer F.Cu) (net 1) (status 400000))
+  (segment (start 76.2 98.2) (end 75.5 97.5) (width 0.5) (layer F.Cu) (net 1))
+  (via (at 75.5 97.5) (size 0.6) (drill 0.4) (layers F.Cu B.Cu) (net 1))
+  (segment (start 150.5 102.5) (end 150.5 100.5) (width 1) (layer F.Cu) (net 1))
+  (via (at 150.5 100.5) (size 0.8) (drill 0.6) (layers F.Cu B.Cu) (net 1))
+  (segment (start 150.5 104.5) (end 150.5 102.5) (width 1) (layer F.Cu) (net 1))
+  (via (at 150.5 102.5) (size 0.8) (drill 0.6) (layers F.Cu B.Cu) (net 1))
+  (segment (start 150.495 106.77) (end 150.495 104.505) (width 1) (layer F.Cu) (net 1) (status 400000))
+  (segment (start 150.495 104.505) (end 150.5 104.5) (width 1) (layer F.Cu) (net 1))
+  (via (at 150.5 104.5) (size 0.8) (drill 0.6) (layers F.Cu B.Cu) (net 1))
+  (segment (start 155.5 102.5) (end 155.5 100.5) (width 1) (layer F.Cu) (net 1))
+  (via (at 155.5 100.5) (size 0.8) (drill 0.6) (layers F.Cu B.Cu) (net 1))
+  (segment (start 155.5 104.5) (end 155.5 102.5) (width 1) (layer F.Cu) (net 1))
+  (via (at 155.5 102.5) (size 0.8) (drill 0.6) (layers F.Cu B.Cu) (net 1))
+  (segment (start 155.575 106.77) (end 155.575 104.575) (width 1) (layer F.Cu) (net 1) (status 400000))
+  (segment (start 155.575 104.575) (end 155.5 104.5) (width 1) (layer F.Cu) (net 1))
+  (via (at 155.5 104.5) (size 0.8) (drill 0.6) (layers F.Cu B.Cu) (net 1))
+  (segment (start 107.5 103.5) (end 107.5 105) (width 1) (layer F.Cu) (net 1))
+  (segment (start 107.5 105) (end 106.5 106) (width 1) (layer F.Cu) (net 1))
+  (via (at 106.5 106) (size 0.8) (drill 0.6) (layers F.Cu B.Cu) (net 1))
+  (segment (start 109.5 103.5) (end 107.5 103.5) (width 1) (layer F.Cu) (net 1))
+  (via (at 107.5 103.5) (size 0.8) (drill 0.6) (layers F.Cu B.Cu) (net 1))
+  (segment (start 111.125 103.505) (end 109.505 103.505) (width 1) (layer F.Cu) (net 1) (status 400000))
+  (segment (start 109.505 103.505) (end 109.5 103.5) (width 1) (layer F.Cu) (net 1))
+  (via (at 109.5 103.5) (size 0.8) (drill 0.6) (layers F.Cu B.Cu) (net 1))
+  (segment (start 118.5 80) (end 116.5 80) (width 1) (layer F.Cu) (net 1))
+  (via (at 116.5 80) (size 0.8) (drill 0.6) (layers F.Cu B.Cu) (net 1))
+  (segment (start 120.5 80) (end 118.5 80) (width 1) (layer F.Cu) (net 1))
+  (via (at 118.5 80) (size 0.8) (drill 0.6) (layers F.Cu B.Cu) (net 1))
+  (segment (start 121.285 83.025) (end 121.285 80.785) (width 1) (layer F.Cu) (net 1))
+  (segment (start 121.285 80.785) (end 120.5 80) (width 1) (layer F.Cu) (net 1))
+  (via (at 120.5 80) (size 0.8) (drill 0.6) (layers F.Cu B.Cu) (net 1))
+  (segment (start 104.013 109.855) (end 110.355 109.855) (width 1) (layer F.Cu) (net 1))
+  (segment (start 110.355 109.855) (end 110.5 110) (width 1) (layer F.Cu) (net 1))
+  (via (at 110.5 110) (size 0.8) (drill 0.6) (layers F.Cu B.Cu) (net 1))
+  (segment (start 104.013 109.855) (end 108.355 109.855) (width 1) (layer F.Cu) (net 1))
+  (segment (start 108.355 109.855) (end 108.5 110) (width 1) (layer F.Cu) (net 1))
+  (via (at 108.5 110) (size 0.8) (drill 0.6) (layers F.Cu B.Cu) (net 1))
+  (segment (start 104.013 109.855) (end 106.355 109.855) (width 1) (layer F.Cu) (net 1))
+  (segment (start 106.355 109.855) (end 106.5 110) (width 1) (layer F.Cu) (net 1))
+  (via (at 106.5 110) (size 0.8) (drill 0.6) (layers F.Cu B.Cu) (net 1))
+  (segment (start 111.5 105) (end 110 105) (width 0.5) (layer F.Cu) (net 1))
+  (via (at 110 105) (size 0.6) (drill 0.4) (layers F.Cu B.Cu) (net 1))
+  (segment (start 113 105) (end 111.5 105) (width 0.5) (layer F.Cu) (net 1))
+  (via (at 111.5 105) (size 0.6) (drill 0.4) (layers F.Cu B.Cu) (net 1))
+  (segment (start 114.5 105) (end 113 105) (width 0.5) (layer F.Cu) (net 1))
+  (via (at 113 105) (size 0.6) (drill 0.4) (layers F.Cu B.Cu) (net 1))
+  (segment (start 116 105) (end 114.5 105) (width 0.5) (layer F.Cu) (net 1))
+  (via (at 114.5 105) (size 0.6) (drill 0.4) (layers F.Cu B.Cu) (net 1))
+  (segment (start 117.5 105) (end 116 105) (width 0.5) (layer F.Cu) (net 1))
+  (via (at 116 105) (size 0.6) (drill 0.4) (layers F.Cu B.Cu) (net 1))
+  (segment (start 118.11 106.45) (end 118.11 105.61) (width 0.5) (layer F.Cu) (net 1))
+  (segment (start 118.11 105.61) (end 117.5 105) (width 0.5) (layer F.Cu) (net 1))
+  (via (at 117.5 105) (size 0.6) (drill 0.4) (layers F.Cu B.Cu) (net 1))
+  (segment (start 125.5 104) (end 125.5 105.5) (width 0.5) (layer F.Cu) (net 1))
+  (via (at 125.5 105.5) (size 0.6) (drill 0.4) (layers F.Cu B.Cu) (net 1))
+  (segment (start 125.5 102.5) (end 125.5 104) (width 0.5) (layer F.Cu) (net 1))
+  (via (at 125.5 104) (size 0.6) (drill 0.4) (layers F.Cu B.Cu) (net 1))
+  (segment (start 127.32 101.87) (end 126.13 101.87) (width 0.5) (layer F.Cu) (net 1))
+  (segment (start 126.13 101.87) (end 125.5 102.5) (width 0.5) (layer F.Cu) (net 1))
+  (via (at 125.5 102.5) (size 0.6) (drill 0.4) (layers F.Cu B.Cu) (net 1))
+  (segment (start 137 104) (end 137 105.5) (width 0.5) (layer F.Cu) (net 1))
+  (via (at 137 105.5) (size 0.6) (drill 0.4) (layers F.Cu B.Cu) (net 1))
+  (segment (start 137 102.5) (end 137 104) (width 0.5) (layer F.Cu) (net 1))
+  (via (at 137 104) (size 0.6) (drill 0.4) (layers F.Cu B.Cu) (net 1))
+  (segment (start 138.75 101.87) (end 137.63 101.87) (width 0.5) (layer F.Cu) (net 1))
+  (segment (start 137.63 101.87) (end 137 102.5) (width 0.5) (layer F.Cu) (net 1))
+  (via (at 137 102.5) (size 0.6) (drill 0.4) (layers F.Cu B.Cu) (net 1))
+  (segment (start 96.5 93.5) (end 98 93.5) (width 0.7) (layer F.Cu) (net 1))
+  (via (at 98 93.5) (size 0.6) (drill 0.4) (layers F.Cu B.Cu) (net 1))
+  (segment (start 96.5 93.5) (end 96.5 95) (width 0.7) (layer F.Cu) (net 1))
+  (via (at 96.5 95) (size 0.6) (drill 0.4) (layers F.Cu B.Cu) (net 1))
+  (segment (start 96.5 92) (end 96.5 93.5) (width 0.7) (layer F.Cu) (net 1))
+  (via (at 96.5 93.5) (size 0.6) (drill 0.4) (layers F.Cu B.Cu) (net 1))
+  (segment (start 96.52 88.425) (end 96.52 91.98) (width 0.7) (layer F.Cu) (net 1))
+  (segment (start 96.52 91.98) (end 96.5 92) (width 0.7) (layer F.Cu) (net 1))
+  (via (at 96.5 92) (size 0.6) (drill 0.4) (layers F.Cu B.Cu) (net 1))
+  (segment (start 82 85) (end 82 83.5) (width 0.7) (layer F.Cu) (net 1))
+  (via (at 82 83.5) (size 0.6) (drill 0.4) (layers F.Cu B.Cu) (net 1))
+  (segment (start 82 86.5) (end 82 85) (width 0.7) (layer F.Cu) (net 1))
+  (via (at 82 85) (size 0.6) (drill 0.4) (layers F.Cu B.Cu) (net 1))
+  (segment (start 82 88) (end 82 86.5) (width 0.7) (layer F.Cu) (net 1))
+  (via (at 82 86.5) (size 0.6) (drill 0.4) (layers F.Cu B.Cu) (net 1))
+  (segment (start 77.47 88.425) (end 81.575 88.425) (width 0.7) (layer F.Cu) (net 1))
+  (segment (start 81.575 88.425) (end 82 88) (width 0.7) (layer F.Cu) (net 1))
+  (via (at 82 88) (size 0.6) (drill 0.4) (layers F.Cu B.Cu) (net 1))
   (via (at 120.635 65.786) (size 0.6) (drill 0.4) (layers F.Cu B.Cu) (net 1))
   (segment (start 120.635 65.786) (end 120.65 65.786) (width 0.5) (layer B.Cu) (net 1))
@@
   (segment (start 124.079 121.285) (end 126.365 121.285) (width 2) (layer F.Cu) (net 2))
   (segment (start 120.745 117.951) (end 124.079 121.285) (width 2) (layer F.Cu) (net 2))
-  (segment (start 74.295 133.095) (end 77.47 133.095) (width 0.4) (layer F.Cu) (net 3) (status C00000))
+  (segment (start 112.8 75.184) (end 112.8 79.3) (width 0.4) (layer F.Cu) (net 3))
+  (segment (start 112.8 79.3) (end 116 82.5) (width 0.4) (layer F.Cu) (net 3))
+  (segment (start 116 82.5) (end 116 89.5) (width 0.4) (layer F.Cu) (net 3))
+  (segment (start 116 89.5) (end 111.445 94.055) (width 0.4) (layer F.Cu) (net 3))
+  (segment (start 111.445 94.055) (end 111.445 96.52) (width 0.4) (layer F.Cu) (net 3))
+  (segment (start 74.295 133.095) (end 77.47 133.095) (width 0.4) (layer F.Cu) (net 3))
   (segment (start 72.136 96.012) (end 72.136 132.334) (width 0.4) (layer F.Cu) (net 3))
   (segment (start 72.136 132.334) (end 72.897 133.095) (width 0.4) (layer F.Cu) (net 3))
@@
       )
     )
+  )
+  (zone (net 1) (net_name GND) (layer F.Cu) (hatch edge 0.508)
+    (connect_pads (clearance 0.508))
+    (min_thickness 0.254)
+    (fill (arc_segments 16) (thermal_gap 0.508) (thermal_bridge_width 0.508) (smoothing fillet) (radius 0.508))
+    (polygon
+      (pts
+        (xy 159 134.5) (xy 72 134.5) (xy 72 51.5) (xy 159 51.5)
+      )
+    )
+  )
+  (zone (net 1) (net_name GND) (layer B.Cu) (hatch edge 0.508)
+    (connect_pads (clearance 0.508))
+    (min_thickness 0.254)
+    (fill (arc_segments 16) (thermal_gap 0.508) (thermal_bridge_width 0.508) (smoothing fillet) (radius 0.508))
+    (polygon
+      (pts
+        (xy 159 134.5) (xy 72 134.5) (xy 72 51.5) (xy 159 51.5)
+      )
+    )
