File: pcb/antiflood.kicad_pcb (KiCad board)
At the start: 2 copper layers, 88 x 84 mm, 98 parts, among them J1 Barrel_Jack, J10 Screw_Terminal_01x02, J11 Screw_Terminal_01x02, J12 Screw_Terminal_01x02, J13 Screw_Terminal_01x02, J2 Conn_01x03_Male, J3 01x03, J4 01x03, J5 Conn_02x04_Odd_Even, J6 Conn_02x05_Odd_Even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

Commit message: PCB: preprint
Routing:
- net GND: track 123.9 -> 133.8 mm, vias 47 -> 46
- net +5V: track 363.4 -> 354.2 mm
- net /A6: track 159.5 -> 166.2 mm
- net Net-(D8-Pad1): track 27.6 -> 25.7 mm
- net /EPWR: track 43.8 -> 42.0 mm
- net Net-(D1-Pad2): track 91.0 -> 92.2 mm
- net /BTMP: track 38.2 -> 37.4 mm
Other:
- board text added: "ATIFLOOD PROJECT PCB-3"
- board text added: "Copyright 2019 Alexey <Inverse> Shumeiko"
- board text added: "DC 12V"
- board text added: "Main Control Module"
- board text added: "RX IO0 IO2 GND"
- board text added: "Vcc RST EN TX"
- board text removed: "WiFi Antenna"

Commit message: PCB: to production
Routing:
- net /A6: track 166.2 -> 152.5 mm
- net +5V: track 354.2 -> 361.7 mm
Other:
- board text added: "Control"
- board text added: "Module"
- board text added: "Valve"
- board text removed: "Main Control Module"
Changed lines of the file:
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@@
     (area 68.157143 48.874999 162.842858 137.075001)
     (thickness 1.6)
-    (drawings 64)
+    (drawings 66)
     (tracks 845)
     (zones 0)
@@
     (pad_to_mask_clearance 0)
     (aux_axis_origin 71.505 50.975)
-    (visible_elements FFFEF77F)
+    (visible_elements FFFEFF7F)
     (pcbplotparams
       (layerselection 0x00030_80000001)
@@
     (pad 1 thru_hole circle (at 0 0) (size 6.4 6.4) (drill 3.2) (layers *.Cu *.Mask))
   )
+  (gr_text Module (at 143 97) (layer F.SilkS)
+    (effects (font (size 3 3) (thickness 0.4)))
+  )
+  (gr_text Control (at 143 92) (layer F.SilkS)
+    (effects (font (size 3 3) (thickness 0.4)))
+  )
   (gr_text "Copyright 2019\nAlexey <Inverse> Shumeiko" (at 131.826 94.742) (layer B.SilkS)
     (effects (font (size 2 2) (thickness 0.25) italic) (justify mirror))
@@
     (effects (font (size 1.5 1.5) (thickness 0.3)))
   )
-  (gr_text "Main Control\nModule" (at 142.24 93.472) (layer F.SilkS)
+  (gr_text Valve (at 141 87) (layer F.SilkS)
     (effects (font (size 3 3) (thickness 0.4)))
   )
@@
   (segment (start 124.079 121.285) (end 126.365 121.285) (width 2) (layer F.Cu) (net 2))
   (segment (start 120.745 117.951) (end 124.079 121.285) (width 2) (layer F.Cu) (net 2))
+  (segment (start 72.136 96.012) (end 72.136 132.334) (width 0.4) (layer F.Cu) (net 3))
+  (segment (start 72.136 96.012) (end 72.136 93.472) (width 0.5) (layer F.Cu) (net 3))
+  (segment (start 72.897 133.095) (end 77.47 133.095) (width 0.4) (layer F.Cu) (net 3))
+  (segment (start 72.136 132.334) (end 72.897 133.095) (width 0.4) (layer F.Cu) (net 3))
+  (segment (start 73.66 96.2) (end 72.136 96.2) (width 0.4) (layer F.Cu) (net 3))
+  (segment (start 72.136 96.2) (end 72.136 96.266) (width 0.4) (layer F.Cu) (net 3))
+  (segment (start 72.136 93.472) (end 72.136 96.266) (width 0.7) (layer F.Cu) (net 3))
+  (segment (start 72.136 96.266) (end 72.136 99.06) (width 0.7) (layer F.Cu) (net 3))
+  (segment (start 72.136 99.06) (end 74.93 99.06) (width 0.7) (layer F.Cu) (net 3))
+  (segment (start 89.295 88.875) (end 89.295 90.791) (width 0.7) (layer F.Cu) (net 3))
+  (segment (start 89.295 90.791) (end 88.9 91.186) (width 0.7) (layer F.Cu) (net 3))
+  (segment (start 88.9 91.186) (end 74.422 91.186) (width 0.7) (layer F.Cu) (net 3))
+  (segment (start 74.422 91.186) (end 72.136 93.472) (width 0.7) (layer F.Cu) (net 3))
   (segment (start 123.035 61.711) (end 123.035 60.043) (width 0.5) (layer F.Cu) (net 3))
   (segment (start 123.035 60.043) (end 122.936 59.944) (width 0.5) (layer F.Cu) (net 3))
@@
   (segment (start 111.445 94.055) (end 111.445 96.52) (width 0.4) (layer F.Cu) (net 3))
   (segment (start 74.295 133.095) (end 77.47 133.095) (width 0.4) (layer F.Cu) (net 3))
-  (segment (start 72.136 96.012) (end 72.136 132.334) (width 0.4) (layer F.Cu) (net 3))
-  (segment (start 72.136 132.334) (end 72.897 133.095) (width 0.4) (layer F.Cu) (net 3))
-  (segment (start 72.897 133.095) (end 77.47 133.095) (width 0.4) (layer F.Cu) (net 3))
   (segment (start 123.444 77.47) (end 121.158 77.47) (width 0.7) (layer F.Cu) (net 3))
   (segment (start 121.158 77.47) (end 121.5 77.47) (width 0.7) (layer F.Cu) (net 3))
@@
   (segment (start 127.635 113.665) (end 126.365 113.665) (width 0.5) (layer F.Cu) (net 3))
   (segment (start 128.81 112.49) (end 127.635 113.665) (width 0.5) (layer F.Cu) (net 3))
-  (segment (start 73.66 96.2) (end 72.324 96.2) (width 0.5) (layer F.Cu) (net 3))
   (segment (start 89.295 90.791) (end 89.295 88.875) (width 0.5) (layer F.Cu) (net 3))
   (segment (start 88.9 91.186) (end 89.295 90.791) (width 0.5) (layer F.Cu) (net 3))
-  (segment (start 74.422 91.186) (end 88.9 91.186) (width 0.5) (layer F.Cu) (net 3))
-  (segment (start 72.136 93.472) (end 74.422 91.186) (width 0.5) (layer F.Cu) (net 3))
-  (segment (start 72.136 96.012) (end 72.136 93.472) (width 0.5) (layer F.Cu) (net 3))
-  (segment (start 72.324 96.2) (end 72.136 96.012) (width 0.5) (layer F.Cu) (net 3))
-  (segment (start 74.93 99.06) (end 74.93 98.552) (width 0.5) (layer F.Cu) (net 3))
-  (segment (start 74.93 98.552) (end 73.66 97.282) (width 0.5) (layer F.Cu) (net 3))
-  (segment (start 73.66 97.282) (end 73.66 96.2) (width 0.5) (layer F.Cu) (net 3))
   (segment (start 103.762 85.852) (end 103.635 85.725) (width 0.4) (layer F.Cu) (net 3))
   (segment (start 103.635 85.725) (end 101.473 85.725) (width 2) (layer F.Cu) (net 3))
@@
   (segment (start 118.11 78.486) (end 117.348 77.724) (width 0.4) (layer F.Cu) (net 12))
   (segment (start 120.142 78.486) (end 118.486 78.486) (width 0.4) (layer F.Cu) (net 12))
-  (segment (start 116.84 64.77) (end 121.666 59.944) (width 0.4) (layer B.Cu) (net 12))
   (segment (start 124.968 98.806) (end 124.968 80.772) (width 0.4) (layer F.Cu) (net 12))
   (segment (start 124.968 80.772) (end 122.682 78.486) (width 0.4) (layer F.Cu) (net 12))
   (segment (start 122.682 78.486) (end 120.142 78.486) (width 0.4) (layer F.Cu) (net 12))
-  (segment (start 116.84 64.77) (end 121.666 59.944) (width 0.4) (layer B.Cu) (net 12))
   (via (at 121.666 59.944) (size 0.6) (drill 0.4) (layers F.Cu B.Cu) (net 12))
   (segment (start 122.235 60.513) (end 122.235 61.711) (width 0.4) (layer F.Cu) (net 12))
